Commit message: add lidars

File: autoware_vehicle/urdf/sensor_kit.xacro (robot description, xacro)
@@ -20,179 +20,208 @@
     <xacro:property name="calibration" value="${xacro.load_yaml('$(arg config_dir)/sensor_kit_calibration.yaml')}"/>
     <!-- lidar -->
-    <xacro:VLS-128 parent="sensor_kit_base_link" name="velodyne_top" topic="/points_raw" hz="10" samples="220" gpu="$(arg gpu)">
-      <origin
-        xyz="${calibration['sensor_kit_base_link']['velodyne_top_base_link']['x']}
-             ${calibration['sensor_kit_base_link']['velodyne_top_base_link']['y']}
-             ${calibration['sensor_kit_base_link']['velodyne_top_base_link']['z']}"
-        rpy="${calibration['sensor_kit_base_link']['velodyne_top_base_link']['roll']}
-             ${calibration['sensor_kit_base_link']['velodyne_top_base_link']['pitch']}
-             ${calibration['sensor_kit_base_link']['velodyne_top_base_link']['yaw']}"
+    <xacro:VLS-128 parent="sensor_kit_base_link" name="VLS128_TOP" topic="/points_raw" hz="10" samples="220" gpu="$(arg gpu)">
+      <origin
+        xyz="${calibration['sensor_kit_base_link']['VLS128_TOP_base_link']['x']}
+             ${calibration['sensor_kit_base_link']['VLS128_TOP_base_link']['y']}
+             ${calibration['sensor_kit_base_link']['VLS128_TOP_base_link']['z']}"
+        rpy="${calibration['sensor_kit_base_link']['VLS128_TOP_base_link']['roll']}
+             ${calibration['sensor_kit_base_link']['VLS128_TOP_base_link']['pitch']}
+             ${calibration['sensor_kit_base_link']['VLS128_TOP_base_link']['yaw']}"
       />
     </xacro:VLS-128>
-    <xacro:VLP-16 parent="sensor_kit_base_link" name="velodyne_left" topic="/points_raw" hz="10" samples="220" gpu="$(arg gpu)">
-      <origin
-        xyz="${calibration['sensor_kit_base_link']['velodyne_left_base_link']['x']}
-             ${calibration['sensor_kit_base_link']['velodyne_left_base_link']['y']}
-             ${calibration['sensor_kit_base_link']['velodyne_left_base_link']['z']}"
-        rpy="${calibration['sensor_kit_base_link']['velodyne_left_base_link']['roll']}
-             ${calibration['sensor_kit_base_link']['velodyne_left_base_link']['pitch']}
-             ${calibration['sensor_kit_base_link']['velodyne_left_base_link']['yaw']}"
-      />
-    </xacro:VLP-16>
-    <xacro:VLP-16 parent="sensor_kit_base_link" name="velodyne_right" topic="/points_raw" hz="10" samples="220" gpu="$(arg gpu)">
-      <origin
-        xyz="${calibration['sensor_kit_base_link']['velodyne_right_base_link']['x']}
-             ${calibration['sensor_kit_base_link']['velodyne_right_base_link']['y']}
-             ${calibration['sensor_kit_base_link']['velodyne_right_base_link']['z']}"
-        rpy="${calibration['sensor_kit_base_link']['velodyne_right_base_link']['roll']}
-             ${calibration['sensor_kit_base_link']['velodyne_right_base_link']['pitch']}
-             ${calibration['sensor_kit_base_link']['velodyne_right_base_link']['yaw']}"
+    <xacro:VLP-16 parent="sensor_kit_base_link" name="VLP16_BL" topic="/points_raw" hz="10" samples="220" gpu="$(arg gpu)">
+      <origin
+        xyz="${calibration['sensor_kit_base_link']['VLP16_BL_base_link']['x']}
+             ${calibration['sensor_kit_base_link']['VLP16_BL_base_link']['y']}
+             ${calibration['sensor_kit_base_link']['VLP16_BL_base_link']['z']}"
+        rpy="${calibration['sensor_kit_base_link']['VLP16_BL_base_link']['roll']}
+             ${calibration['sensor_kit_base_link']['VLP16_BL_base_link']['pitch']}
+             ${calibration['sensor_kit_base_link']['VLP16_BL_base_link']['yaw']}"
+      />
+    </xacro:VLP-16>
+    <xacro:VLP-16 parent="sensor_kit_base_link" name="VLP16_BR" topic="/points_raw" hz="10" samples="220" gpu="$(arg gpu)">
+      <origin
+        xyz="${calibration['sensor_kit_base_link']['VLP16_BR_base_link']['x']}
+             ${calibration['sensor_kit_base_link']['VLP16_BR_base_link']['y']}
+             ${calibration['sensor_kit_base_link']['VLP16_BR_base_link']['z']}"
+        rpy="${calibration['sensor_kit_base_link']['VLP16_BR_base_link']['roll']}
+             ${calibration['sensor_kit_base_link']['VLP16_BR_base_link']['pitch']}
+             ${calibration['sensor_kit_base_link']['VLP16_BR_base_link']['yaw']}"
+      />
+    </xacro:VLP-16>
+    <xacro:VLP-16 parent="sensor_kit_base_link" name="VLP16_ML" topic="/points_raw" hz="10" samples="220" gpu="$(arg gpu)">
+      <origin
+        xyz="${calibration['sensor_kit_base_link']['VLP16_ML_base_link']['x']}
+             ${calibration['sensor_kit_base_link']['VLP16_ML_base_link']['y']}
+             ${calibration['sensor_kit_base_link']['VLP16_ML_base_link']['z']}"
+        rpy="${calibration['sensor_kit_base_link']['VLP16_ML_base_link']['roll']}
+             ${calibration['sensor_kit_base_link']['VLP16_ML_base_link']['pitch']}
+             ${calibration['sensor_kit_base_link']['VLP16_ML_base_link']['yaw']}"
+      />
+    </xacro:VLP-16>
+    <xacro:VLP-16 parent="sensor_kit_base_link" name="VLP16_MR" topic="/points_raw" hz="10" samples="220" gpu="$(arg gpu)">
+      <origin
+        xyz="${calibration['sensor_kit_base_link']['VLP16_MR_base_link']['x']}
+             ${calibration['sensor_kit_base_link']['VLP16_MR_base_link']['y']}
+             ${calibration['sensor_kit_base_link']['VLP16_MR_base_link']['z']}"
+        rpy="${calibration['sensor_kit_base_link']['VLP16_MR_base_link']['roll']}
+             ${calibration['sensor_kit_base_link']['VLP16_MR_base_link']['pitch']}
+             ${calibration['sensor_kit_base_link']['VLP16_MR_base_link']['yaw']}"
+      />
+    </xacro:VLP-16>
+    <xacro:VLP-16 parent="sensor_kit_base_link" name="RS_BPEARL_F" topic="/points_raw" hz="10" samples="220" gpu="$(arg gpu)">
+      <origin
+        xyz="${calibration['sensor_kit_base_link']['RS_BPEARL_F_base_link']['x']}
+             ${calibration['sensor_kit_base_link']['RS_BPEARL_F_base_link']['y']}
+             ${calibration['sensor_kit_base_link']['RS_BPEARL_F_base_link']['z']}"
+        rpy="${calibration['sensor_kit_base_link']['RS_BPEARL_F_base_link']['roll']}
+             ${calibration['sensor_kit_base_link']['RS_BPEARL_F_base_link']['pitch']}
+             ${calibration['sensor_kit_base_link']['RS_BPEARL_F_base_link']['yaw']}"
       />
     </xacro:VLP-16>
     <!-- camera -->
     <xacro:monocular_camera_macro
-      name="traffic_light_right_camera/camera"
-      parent="sensor_kit_base_link"
-      namespace=""
-      x="${calibration['sensor_kit_base_link']['traffic_light_right_camera/camera_link']['x']}"
-      y="${calibration['sensor_kit_base_link']['traffic_light_right_camera/camera_link']['y']}"
-      z="${calibration['sensor_kit_base_link']['traffic_light_right_camera/camera_link']['z']}"
-      roll="${calibration['sensor_kit_base_link']['traffic_light_right_camera/camera_link']['roll']}"
-      pitch="${calibration['sensor_kit_base_link']['traffic_light_right_camera/camera_link']['pitch']}"
-      yaw="${calibration['sensor_kit_base_link']['traffic_light_right_camera/camera_link']['yaw']}"
-      fps="30"
-      width="800"
-      height="400"
-      fov="1.3"
-    />
-    <xacro:monocular_camera_macro
-      name="traffic_light_left_camera/camera"
-      parent="sensor_kit_base_link"
-      namespace=""
-      x="${calibration['sensor_kit_base_link']['traffic_light_left_camera/camera_link']['x']}"
-      y="${calibration['sensor_kit_base_link']['traffic_light_left_camera/camera_link']['y']}"
-      z="${calibration['sensor_kit_base_link']['traffic_light_left_camera/camera_link']['z']}"
-      roll="${calibration['sensor_kit_base_link']['traffic_light_left_camera/camera_link']['roll']}"
-      pitch="${calibration['sensor_kit_base_link']['traffic_light_left_camera/camera_link']['pitch']}"
-      yaw="${calibration['sensor_kit_base_link']['traffic_light_left_camera/camera_link']['yaw']}"
-      fps="30"
-      width="800"
-      height="400"
-      fov="1.3"
-    />
-    <xacro:monocular_camera_macro
-      name="camera0/camera"
-      parent="sensor_kit_base_link"
-      namespace=""
-      x="${calibration['sensor_kit_base_link']['camera0/camera_link']['x']}"
-      y="${calibration['sensor_kit_base_link']['camera0/camera_link']['y']}"
-      z="${calibration['sensor_kit_base_link']['camera0/camera_link']['z']}"
-      roll="${calibration['sensor_kit_base_link']['camera0/camera_link']['roll']}"
-      pitch="${calibration['sensor_kit_base_link']['camera0/camera_link']['pitch']}"
-      yaw="${calibration['sensor_kit_base_link']['camera0/camera_link']['yaw']}"
-      fps="30"
-      width="800"
-      height="400"
-      fov="1.3"
-    />
-    <xacro:monocular_camera_macro
-      name="camera1/camera"
-      parent="sensor_kit_base_link"
-      namespace=""
-      x="${calibration['sensor_kit_base_link']['camera1/camera_link']['x']}"
-      y="${calibration['sensor_kit_base_link']['camera1/camera_link']['y']}"
-      z="${calibration['sensor_kit_base_link']['camera1/camera_link']['z']}"
-      roll="${calibration['sensor_kit_base_link']['camera1/camera_link']['roll']}"
-      pitch="${calibration['sensor_kit_base_link']['camera1/camera_link']['pitch']}"
-      yaw="${calibration['sensor_kit_base_link']['camera1/camera_link']['yaw']}"
-      fps="30"
-      width="800"
-      height="400"
-      fov="1.3"
-    />
-    <xacro:monocular_camera_macro
-      name="camera2/camera"
-      parent="sensor_kit_base_link"
-      namespace=""
-      x="${calibration['sensor_kit_base_link']['camera2/camera_link']['x']}"
-      y="${calibration['sensor_kit_base_link']['camera2/camera_link']['y']}"
-      z="${calibration['sensor_kit_base_link']['camera2/camera_link']['z']}"
-      roll="${calibration['sensor_kit_base_link']['camera2/camera_link']['roll']}"
-      pitch="${calibration['sensor_kit_base_link']['camera2/camera_link']['pitch']}"
-      yaw="${calibration['sensor_kit_base_link']['camera2/camera_link']['yaw']}"
-      fps="30"
-      width="800"
-      height="400"
-      fov="1.3"
-    />
-    <xacro:monocular_camera_macro
-      name="camera3/camera"
-      parent="sensor_kit_base_link"
-      namespace=""
-      x="${calibration['sensor_kit_base_link']['camera3/camera_link']['x']}"
-      y="${calibration['sensor_kit_base_link']['camera3/camera_link']['y']}"
-      z="${calibration['sensor_kit_base_link']['camera3/camera_link']['z']}"
-      roll="${calibration['sensor_kit_base_link']['camera3/camera_link']['roll']}"
-      pitch="${calibration['sensor_kit_base_link']['camera3/camera_link']['pitch']}"
-      yaw="${calibration['sensor_kit_base_link']['camera3/camera_link']['yaw']}"
-      fps="30"
-      width="800"
-      height="400"
-      fov="1.3"
-    />
-    <xacro:monocular_camera_macro
-      name="camera4/camera"
-      parent="sensor_kit_base_link"
-      namespace=""
-      x="${calibration['sensor_kit_base_link']['camera4/camera_link']['x']}"
-      y="${calibration['sensor_kit_base_link']['camera4/camera_link']['y']}"
-      z="${calibration['sensor_kit_base_link']['camera4/camera_link']['z']}"
-      roll="${calibration['sensor_kit_base_link']['camera4/camera_link']['roll']}"
-      pitch="${calibration['sensor_kit_base_link']['camera4/camera_link']['pitch']}"
-      yaw="${calibration['sensor_kit_base_link']['camera4/camera_link']['yaw']}"
-      fps="30"
-      width="800"
-      height="400"
-      fov="1.3"
-    />
-    <xacro:monocular_camera_macro
-      name="camera5/camera"
-      parent="sensor_kit_base_link"
-      namespace=""
-      x="${calibration['sensor_kit_base_link']['camera5/camera_link']['x']}"
-      y="${calibration['sensor_kit_base_link']['camera5/camera_link']['y']}"
-      z="${calibration['sensor_kit_base_link']['camera5/camera_link']['z']}"
-      roll="${calibration['sensor_kit_base_link']['camera5/camera_link']['roll']}"
-      pitch="${calibration['sensor_kit_base_link']['camera5/camera_link']['pitch']}"
-      yaw="${calibration['sensor_kit_base_link']['camera5/camera_link']['yaw']}"
-      fps="30"
-      width="800"
-      height="400"
-      fov="1.3"
-    />
-    <!-- gnss -->
+      name="CAM_FR/camera"
+      parent="sensor_kit_base_link"
+      namespace=""
+      x="${calibration['sensor_kit_base_link']['CAM_FR/camera_link']['x']}"
+      y="${calibration['sensor_kit_base_link']['CAM_FR/camera_link']['y']}"
+      z="${calibration['sensor_kit_base_link']['CAM_FR/camera_link']['z']}"
+      roll="${calibration['sensor_kit_base_link']['CAM_FR/camera_link']['roll']}"
+      pitch="${calibration['sensor_kit_base_link']['CAM_FR/camera_link']['pitch']}"
+      yaw="${calibration['sensor_kit_base_link']['CAM_FR/camera_link']['yaw']}"
+      fps="30"
+      width="800"
+      height="400"
+      fov="1.3"
+    />
+    <xacro:monocular_camera_macro
+      name="CAM_F/camera"
+      parent="sensor_kit_base_link"
+      namespace=""
+      x="${calibration['sensor_kit_base_link']['CAM_F/camera_link']['x']}"
+      y="${calibration['sensor_kit_base_link']['CAM_F/camera_link']['y']}"
+      z="${calibration['sensor_kit_base_link']['CAM_F/camera_link']['z']}"
+      roll="${calibration['sensor_kit_base_link']['CAM_F/camera_link']['roll']}"
+      pitch="${calibration['sensor_kit_base_link']['CAM_F/camera_link']['pitch']}"
+      yaw="${calibration['sensor_kit_base_link']['CAM_F/camera_link']['yaw']}"
+      fps="30"
+      width="800"
+      height="400"
+      fov="1.3"
+    />
+    <xacro:monocular_camera_macro
+      name="CAM_FL/camera"
+      parent="sensor_kit_base_link"
+      namespace=""
+      x="${calibration['sensor_kit_base_link']['CAM_FL/camera_link']['x']}"
+      y="${calibration['sensor_kit_base_link']['CAM_FL/camera_link']['y']}"
+      z="${calibration['sensor_kit_base_link']['CAM_FL/camera_link']['z']}"
+      roll="${calibration['sensor_kit_base_link']['CAM_FL/camera_link']['roll']}"
+      pitch="${calibration['sensor_kit_base_link']['CAM_FL/camera_link']['pitch']}"
+      yaw="${calibration['sensor_kit_base_link']['CAM_FL/camera_link']['yaw']}"
+      fps="30"
+      width="800"
+      height="400"
+      fov="1.3"
+    />
+    <xacro:monocular_camera_macro
+      name="CAM_ML/camera"
+      parent="sensor_kit_base_link"
+      namespace=""
+      x="${calibration['sensor_kit_base_link']['CAM_ML/camera_link']['x']}"
+      y="${calibration['sensor_kit_base_link']['CAM_ML/camera_link']['y']}"
+      z="${calibration['sensor_kit_base_link']['CAM_ML/camera_link']['z']}"
+      roll="${calibration['sensor_kit_base_link']['CAM_ML/camera_link']['roll']}"
+      pitch="${calibration['sensor_kit_base_link']['CAM_ML/camera_link']['pitch']}"
+      yaw="${calibration['sensor_kit_base_link']['CAM_ML/camera_link']['yaw']}"
+      fps="30"
+      width="800"
+      height="400"
+      fov="1.3"
+    />
+    <xacro:monocular_camera_macro
+      name="CAM_BL/camera"
+      parent="sensor_kit_base_link"
+      namespace=""
+      x="${calibration['sensor_kit_base_link']['CAM_BL/camera_link']['x']}"
+      y="${calibration['sensor_kit_base_link']['CAM_BL/camera_link']['y']}"
+      z="${calibration['sensor_kit_base_link']['CAM_BL/camera_link']['z']}"
+      roll="${calibration['sensor_kit_base_link']['CAM_BL/camera_link']['roll']}"
+      pitch="${calibration['sensor_kit_base_link']['CAM_BL/camera_link']['pitch']}"
+      yaw="${calibration['sensor_kit_base_link']['CAM_BL/camera_link']['yaw']}"
+      fps="30"
+      width="800"
+      height="400"
+      fov="1.3"
+    />
+    <xacro:monocular_camera_macro
+      name="CAM_B/camera"
+      parent="sensor_kit_base_link"
+      namespace=""
+      x="${calibration['sensor_kit_base_link']['CAM_B/camera_link']['x']}"
+      y="${calibration['sensor_kit_base_link']['CAM_B/camera_link']['y']}"
+      z="${calibration['sensor_kit_base_link']['CAM_B/camera_link']['z']}"
+      roll="${calibration['sensor_kit_base_link']['CAM_B/camera_link']['roll']}"
+      pitch="${calibration['sensor_kit_base_link']['CAM_B/camera_link']['pitch']}"
+      yaw="${calibration['sensor_kit_base_link']['CAM_B/camera_link']['yaw']}"
+      fps="30"
+      width="800"
+      height="400"
+      fov="1.3"
+    />
+    <xacro:monocular_camera_macro
+      name="CAM_BR/camera"
+      parent="sensor_kit_base_link"
+      namespace=""
+      x="${calibration['sensor_kit_base_link']['CAM_BR/camera_link']['x']}"
+      y="${calibration['sensor_kit_base_link']['CAM_BR/camera_link']['y']}"
+      z="${calibration['sensor_kit_base_link']['CAM_BR/camera_link']['z']}"
+      roll="${calibration['sensor_kit_base_link']['CAM_BR/camera_link']['roll']}"
+      pitch="${calibration['sensor_kit_base_link']['CAM_BR/camera_link']['pitch']}"
+      yaw="${calibration['sensor_kit_base_link']['CAM_BR/camera_link']['yaw']}"
+      fps="30"
+      width="800"
+      height="400"
+      fov="1.3"
+    />
+    <xacro:monocular_camera_macro
+      name="CAM_MR/camera"
+      parent="sensor_kit_base_link"
+      namespace=""
+      x="${calibration['sensor_kit_base_link']['CAM_MR/camera_link']['x']}"
+      y="${calibration['sensor_kit_base_link']['CAM_MR/camera_link']['y']}"
+      z="${calibration['sensor_kit_base_link']['CAM_MR/camera_link']['z']}"
+      roll="${calibration['sensor_kit_base_link']['CAM_MR/camera_link']['roll']}"
+      pitch="${calibration['sensor_kit_base_link']['CAM_MR/camera_link']['pitch']}"
+      yaw="${calibration['sensor_kit_base_link']['CAM_MR/camera_link']['yaw']}"
+      fps="30"
+      width="800"
+      height="400"
+      fov="1.3"
+    />
+    <!-- gnss-ins -->
     <xacro:imu_macro
-      name="gnss"
-      parent="sensor_kit_base_link"
-      namespace=""
-      x="${calibration['sensor_kit_base_link']['gnss_link']['x']}"
-      y="${calibration['sensor_kit_base_link']['gnss_link']['y']}"
-      z="${calibration['sensor_kit_base_link']['gnss_link']['z']}"
-      roll="${calibration['sensor_kit_base_link']['gnss_link']['roll']}"
-      pitch="${calibration['sensor_kit_base_link']['gnss_link']['pitch']}"
-      yaw="${calibration['sensor_kit_base_link']['gnss_link']['yaw']}"
+      name="GNSS_INS"
+      parent="sensor_kit_base_link"
+      namespace=""
+      x="${calibration['sensor_kit_base_link']['GNSS_INS']['x']}"
+      y="${calibration['sensor_kit_base_link']['GNSS_INS']['y']}"
+      z="${calibration['sensor_kit_base_link']['GNSS_INS']['z']}"
+      roll="${calibration['sensor_kit_base_link']['GNSS_INS']['roll']}"
+      pitch="${calibration['sensor_kit_base_link']['GNSS_INS']['pitch']}"
+      yaw="${calibration['sensor_kit_base_link']['GNSS_INS']['yaw']}"
       fps="100"
     />
-    <!-- imu -->
     <xacro:imu_macro
-      name="tamagawa/imu"
-      parent="sensor_kit_base_link"
-      namespace=""
-      x="${calibration['sensor_kit_base_link']['tamagawa/imu_link']['x']}"
-      y="${calibration['sensor_kit_base_link']['tamagawa/imu_link']['y']}"
-      z="${calibration['sensor_kit_base_link']['tamagawa/imu_link']['z']}"
-      roll="${calibration['sensor_kit_base_link']['tamagawa/imu_link']['roll']}"
-      pitch="${calibration['sensor_kit_base_link']['tamagawa/imu_link']['pitch']}"
-      yaw="${calibration['sensor_kit_base_link']['tamagawa/imu_link']['yaw']}"
+      name="GNSS_INS/gnss_ins"
+      parent="sensor_kit_base_link"
+      namespace=""
+      x="${calibration['sensor_kit_base_link']['GNSS_INS/gnss_ins_link']['x']}"
+      y="${calibration['sensor_kit_base_link']['GNSS_INS/gnss_ins_link']['y']}"
+      z="${calibration['sensor_kit_base_link']['GNSS_INS/gnss_ins_link']['z']}"
+      roll="${calibration['sensor_kit_base_link']['GNSS_INS/gnss_ins_link']['roll']}"
+      pitch="${calibration['sensor_kit_base_link']['GNSS_INS/gnss_ins_link']['pitch']}"
+      yaw="${calibration['sensor_kit_base_link']['GNSS_INS/gnss_ins_link']['yaw']}"
       fps="100"
     />

File: autoware_vehicle/urdf/sensors.xacro (robot description, xacro)
@@ -14,15 +14,3 @@
     yaw="${calibration['base_link']['sensor_kit_base_link']['yaw']}"
   />
-  <!-- embedded sensors -->
-  <xacro:include filename="$(find velodyne_description)/urdf/VLP-16.urdf.xacro"/>
-  <xacro:VLP-16 parent="base_link" name="velodyne_rear" topic="velodyne_rear/velodyne_points" hz="10" samples="220" gpu="false">
-    <origin
-      xyz="${calibration['base_link']['velodyne_rear_base_link']['x']}
-           ${calibration['base_link']['velodyne_rear_base_link']['y']}
-           ${calibration['base_link']['velodyne_rear_base_link']['z']}"
-      rpy="${calibration['base_link']['velodyne_rear_base_link']['roll']}
-           ${calibration['base_link']['velodyne_rear_base_link']['pitch']}
-           ${calibration['base_link']['velodyne_rear_base_link']['yaw']}"
-    />
-  </xacro:VLP-16>
 </robot>

File: autoware_vehicle/urdf/vehicle.xacro (robot description, xacro)
@@ -6,7 +6,8 @@
   <link name="base_link">
     <visual>
-      <origin xyz="${vehicle_info['/**']['ros__parameters']['wheel_base']/2.0} 0 0" rpy="${pi/2.0} 0 ${pi}"/>
+<!--      <origin xyz="${vehicle_info['/**']['ros__parameters']['wheel_base']/2.0} 0 0" rpy="${pi/2.0} 0 ${pi}"/>-->
+      <origin xyz="1.3772 0.0 0.0" rpy="0 0 ${pi/2.0}"/>
       <geometry>
-        <mesh filename="package://autoware_vehicle/mesh/lexus.dae" scale="1 1 1"/>
+        <mesh filename="package://autoware_vehicle/mesh/golf.dae" scale="1 1 1"/>
       </geometry>
     </visual>
