Commit message: fix(vehicle.xacro): fix position

File: autoware_vehicle/urdf/vehicle.xacro (robot description, xacro)
@@ -7,5 +7,5 @@
     <visual>
 <!--      <origin xyz="${vehicle_info['/**']['ros__parameters']['wheel_base']/2.0} 0 0" rpy="${pi/2.0} 0 ${pi}"/>-->
-      <origin xyz="1.3772 0.0 0.0" rpy="0 0 ${pi/2.0}"/>
+      <origin xyz="1.364 0.08 -0.08" rpy="0 0 ${pi/2.0}"/>
       <geometry>
         <mesh filename="package://autoware_vehicle/mesh/golf.dae" scale="1 1 1"/>
